Commit message: Add docking, cart towing, GS capture tools and simulated docking world
- amr_docking: ArUco detector, charger docking via Nav2 docking_server,
  cart reverse docking with hitch-current coupling check, towing mode
  (robot+cart footprint, cart cloud filter, MPPI towing limits, passive
  hitch yaw), printable markers.
- amr_capture: Gaussian Splatting capture rig recording (ZED 2, Mid-360,
  T265), operator crop filter, FAST-LIO config, bag -> COLMAP/nerfstudio
  export with floor alignment, lidar map -> collision mesh.
- amr_isaac: docking world (platform cart with boxes, WiBotic charger,
  indoor GPS, battery, cart latch), custom environments for real-site
  twins (--env-usd, --env-collision), hitch effort as servo drive torque,
  /clock published after TF, demo video tools.
- amr_bringup: docking launch, docking_server and velocity smoother
  settings, filtered lidar cloud.
- amr_hitch: set_yaw_passive service.
- amr_description: WiBotic RC-100 receiver mass.

File: amr_description/urdf/amr_inertials.xacro (robot description, xacro)
@@ -4,7 +4,7 @@
   <xacro:macro name="inertial_base_link">
     <inertial>
-      <origin xyz="-0.00447 -0.00009 0.04774" rpy="0 0 0"/>
-      <mass value="12.8091"/>
-      <inertia ixx="1.304480e-01" ixy="-4.702219e-06" ixz="7.497479e-03" iyy="1.622636e-01" iyz="-2.107030e-04" izz="1.553031e-01"/>
+      <origin xyz="-0.00941 -0.00009 0.04855" rpy="0 0 0"/>
+      <mass value="12.4805"/>
+      <inertia ixx="1.294830e-01" ixy="1.095537e-06" ixz="5.555431e-03" iyy="1.497727e-01" iyz="-2.116543e-04" izz="1.431309e-01"/>
     </inertial>
   </xacro:macro>
